File: hardware/revI/flan36-left.kicad_pcb (KiCad board)
At the start: 2 copper layers, 113.4 x 91.3 mm, 46 parts, among them J1 JST_PH_S2B-PH-K-S, J2 nice!view, K01 KEYSW, K02 KEYSW, K03 KEYSW, K04 KEYSW, K05 KEYSW, K11 KEYSW, K12 KEYSW, K13 KEYSW, K14 KEYSW, K15 KEYSW, K21 KEYSW, K22 KEYSW, K23 KEYSW, K24 KEYSW, K25 KEYSW, K30 KEYSW, K31 KEYSW, K32 KEYSW, SW1 SW_SPDT_PCM12, SW2 SW_SPST_TL3342, U1 nice!nano v2

Commit message: Route revI boards and ship verified ZMK prototype builds
Parts:
- D01, D02, D03, D04, D05, D11, D12, D13, D14, D15, D21, D22, D23, D24, D25, D30, D31, D32: value D_SOD-123 -> 1N4148W
- K01, K02, K03, K04, K05, K11, K12, K13, K14, K15, K21, K22, K23, K24, K25, K30, K31, K32: value KEYSW -> CHOC v1
- SW1: value SW_SPDT_PCM12 -> PCM12SMTR
- SW2: value SW_SPST_TL3342 -> TL3342
Connections:
- net BAT_PLUS renamed /BAT_PLUS
- net BAT_SW renamed /BAT_SW
- net COL0 renamed /COL0
- net COL1 renamed /COL1
- net COL2 renamed /COL2
- net COL3 renamed /COL3
- net COL4 renamed /COL4
- net COL5 renamed /COL5
- net DISP_CS renamed /DISP_CS
- net DISP_MOSI renamed /DISP_MOSI
- net DISP_SCK renamed /DISP_SCK
- net GND renamed /GND
- net K01_A renamed /K01_A
- net K02_A renamed /K02_A
- net K03_A renamed /K03_A
- net K04_A renamed /K04_A
- net K05_A renamed /K05_A
- net K11_A renamed /K11_A
- net K12_A renamed /K12_A
- net K13_A renamed /K13_A
- net K14_A renamed /K14_A
- net K15_A renamed /K15_A
- net K21_A renamed /K21_A
- net K22_A renamed /K22_A
- net K23_A renamed /K23_A
- net K24_A renamed /K24_A
- net K25_A renamed /K25_A
- net K30_A renamed /K30_A
- net K31_A renamed /K31_A
- net K32_A renamed /K32_A
- net RESET renamed /RESET
- net ROW0 renamed /ROW0
- net ROW1 renamed /ROW1
- net ROW2 renamed /ROW2
- net ROW3 renamed /ROW3
- net VCC renamed /VCC
- SW1 pad 3: (no net) -> unconnected-(SW1-C-Pad3)
- U1 pad D15: (no net) -> unconnected-(U1-PadD15)
- U1 pad D18: (no net) -> unconnected-(U1-PadD18)
- U1 pad D19: (no net) -> unconnected-(U1-PadD19)
- U1 pad D20: (no net) -> unconnected-(U1-PadD20)
- U1 pad D21: (no net) -> unconnected-(U1-PadD21)
Routing:
- net /COL1: track 0.00 -> 194.8 mm, vias 0 -> 1
- net /COL2: track 0.00 -> 183.6 mm, vias 0 -> 2
- net /ROW2: track 0.00 -> 160.9 mm, vias 0 -> 1
- net /ROW0: track 0.00 -> 125.6 mm, vias 0 -> 1
- net /COL4: track 0.00 -> 113.1 mm, vias 0 -> 2
- net /ROW1: track 0.00 -> 111.4 mm, vias 0 -> 2
- net /COL3: track 0.00 -> 108.3 mm, vias 0 -> 2
- net /ROW3: track 0.00 -> 107.2 mm, vias 0 -> 3
- net /COL5: track 0.00 -> 101.9 mm, vias 0 -> 2
- net /GND: track 0.00 -> 99.6 mm
- net /COL0: track 0.00 -> 73.7 mm, vias 0 -> 1
- net /RESET: track 0.00 -> 51.7 mm
- net /BAT_SW: track 0.00 -> 45.5 mm, vias 0 -> 1
- net /DISP_SCK: track 0.00 -> 43.7 mm, vias 0 -> 1
- net /DISP_MOSI: track 0.00 -> 38.2 mm, vias 0 -> 1
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Other:
- board text added: "FLAN36 revI - PROTOTYPE"
- board text removed: "FLAN36 revI - UNROUTED"
