File: hardware/revI/flan36-left.kicad_sch (KiCad schematic)
At the start: 41 parts, among them J1 BAT 1S protected, J2 nice!view, K01 CHOC v1, K02 CHOC v1, K03 CHOC v1, K04 CHOC v1, K05 CHOC v1, K11 CHOC v1, K12 CHOC v1, K13 CHOC v1, K14 CHOC v1, K15 CHOC v1, K21 CHOC v1, K22 CHOC v1, K23 CHOC v1, K24 CHOC v1, K25 CHOC v1, K30 CHOC v1, K31 CHOC v1, K32 CHOC v1, SW1 PCM12SMTR, SW2 TL3342, U1 nice!nano v2

Commit message: Lower electronics stack and add flush multicolor frame inlays
Parts:
- J1: value BAT 1S protected -> JST_PH_S2B-PH-K-S; footprint PiantorSlim:Battery_pigtail_2.54 -> PiantorSlim:JST_PH_S2B-PH-K_1x02_P2.00mm_Horizontal

Commit message: Route revI boards and ship verified ZMK prototype builds
Other:
- note added: "FLAN36 revI - LEFT - PROTOTYPE"
- note removed: "FLAN36 revF - LEFT - UNROUTED STUDY"
