File: hardware/revI/flan36-right.kicad_pcb (KiCad board)
At the start: 2 copper layers, 113.4 x 91.3 mm, 46 parts, among them J1 JST_PH_S2B-PH-K-S, J2 nice!view, K01 KEYSW, K02 KEYSW, K03 KEYSW, K04 KEYSW, K05 KEYSW, K11 KEYSW, K12 KEYSW, K13 KEYSW, K14 KEYSW, K15 KEYSW, K21 KEYSW, K22 KEYSW, K23 KEYSW, K24 KEYSW, K25 KEYSW, K30 KEYSW, K31 KEYSW, K32 KEYSW, SW1 SW_SPDT_PCM12, SW2 SW_SPST_TL3342, U1 nice!nano v2

Commit message: Route revI boards and ship verified ZMK prototype builds
Parts:
- D01, D02, D03, D04, D05, D11, D12, D13, D14, D15, D21, D22, D23, D24, D25, D30, D31, D32: value D_SOD-123 -> 1N4148W
- K01, K02, K03, K04, K05, K11, K12, K13, K14, K15, K21, K22, K23, K24, K25, K30, K31, K32: value KEYSW -> CHOC v1
- SW1: value SW_SPDT_PCM12 -> PCM12SMTR
- SW2: value SW_SPST_TL3342 -> TL3342
Connections:
- net BAT_PLUS renamed /BAT_PLUS
- net BAT_SW renamed /BAT_SW
- net COL1 renamed /COL1
- net COL2 renamed /COL2
- net COL3 renamed /COL3
- net COL4 renamed /COL4
- net COL5 renamed /COL5
- net DISP_CS renamed /DISP_CS
- net DISP_MOSI renamed /DISP_MOSI
- net DISP_SCK renamed /DISP_SCK
- net GND renamed /GND
- net K01_A renamed /K01_A
- net K02_A renamed /K02_A
- net K03_A renamed /K03_A
- net K04_A renamed /K04_A
- net K05_A renamed /K05_A
- net K11_A renamed /K11_A
- net K12_A renamed /K12_A
- net K13_A renamed /K13_A
- net K14_A renamed /K14_A
- net K15_A renamed /K15_A
- net K21_A renamed /K21_A
- net K22_A renamed /K22_A
- net K23_A renamed /K23_A
- net K24_A renamed /K24_A
- net K25_A renamed /K25_A
- net K30_A renamed /K30_A
- net K31_A renamed /K31_A
- net K32_A renamed /K32_A
- net RESET renamed /RESET
- net VCC renamed /VCC
- D01 pad 1: ROW0 -> /ROW0
- D02 pad 1: ROW0 -> /ROW0
- D03 pad 1: ROW0 -> /ROW0
- D04 pad 1: ROW0 -> /ROW0
- D05 pad 1: ROW0 -> /ROW0
- D11 pad 1: ROW1 -> /ROW1
- D12 pad 1: ROW1 -> /ROW1
- D13 pad 1: ROW1 -> /ROW1
- D14 pad 1: ROW1 -> /ROW1
- D15 pad 1: ROW1 -> /ROW1
- D21 pad 1: ROW2 -> /ROW2
- D22 pad 1: ROW2 -> /ROW2
- D23 pad 1: ROW2 -> /ROW2
- D24 pad 1: ROW2 -> /ROW2
- D25 pad 1: ROW2 -> /ROW2
- D30 pad 1: ROW3 -> /ROW3
- D31 pad 1: ROW3 -> /ROW3
- D32 pad 1: ROW3 -> /ROW3
- K30 pad 1: COL0 -> /COL0
- SW1 pad 3: (no net) -> unconnected-(SW1-C-Pad3)
- U1 pad D15: (no net) -> /COL0
- U1 pad D18: (no net) -> /ROW3
- U1 pad D19: (no net) -> /ROW2
- U1 pad D2: ROW0 -> unconnected-(U1-PadD2)
- U1 pad D20: (no net) -> /ROW1
- U1 pad D21: (no net) -> /ROW0
- U1 pad D3: ROW1 -> unconnected-(U1-PadD3)
- U1 pad D4: ROW2 -> unconnected-(U1-PadD4)
- U1 pad D5: ROW3 -> unconnected-(U1-PadD5)
- U1 pad D6: COL0 -> unconnected-(U1-PadD6)
Routing:
- net /COL1: track 0.00 -> 198.6 mm, vias 0 -> 3
- net /COL2: track 0.00 -> 198.4 mm, vias 0 -> 1
- net /ROW2: track 0.00 -> 132.1 mm, vias 0 -> 1
- net /COL3: track 0.00 -> 125.1 mm
- net /ROW1: track 0.00 -> 119.8 mm, vias 0 -> 3
- net /ROW0: track 0.00 -> 118.7 mm, vias 0 -> 3
- net /GND: track 0.00 -> 101.4 mm, vias 0 -> 1
- net /COL4: track 0.00 -> 92.3 mm, vias 0 -> 2
- net /ROW3: track 0.00 -> 91.1 mm, vias 0 -> 3
- net /COL0: track 0.00 -> 77.8 mm, vias 0 -> 1
- net /COL5: track 0.00 -> 74.5 mm
- net /BAT_SW: track 0.00 -> 65.0 mm, vias 0 -> 1
- net /RESET: track 0.00 -> 48.8 mm
- net /VCC: track 0.00 -> 36.4 mm, vias 0 -> 1
- net /DISP_MOSI: track 0.00 -> 36.2 mm
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Other:
- board text added: "FLAN36 revI - PROTOTYPE"
- board text removed: "FLAN36 revI - UNROUTED"
